File: _autosave-MCU_Datalogger.kicad_pcb (KiCad board)
At the start: 4 copper layers, 50.5 x 40.2 mm, 29 parts, among them J1 Conn_01x02_Pin, J2 Conn_01x04_Pin, J3 Conn_01x04_Pin, J4 Conn_01x09_Pin, J5 Conn_02x03_Odd_Even, U1 24LC1025, U2 24LC1025, U3 DS1337S_, U4 ATMEGA328P-AU, Y1 32.768kHz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

Commit message: Added README
Routing:
- added copper zone on B.Cu, net GND
- removed copper zone on B.Cu, net /MISO
Changed lines of the file:
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@@
 	)
 	(footprint "Connector_PinHeader_2.54mm:PinHeader_1x04_P2.54mm_Vertical"
-		(locked yes)
 		(layer "F.Cu")
 		(at 125.02 102.89 90)
@@
 		(tags "Through hole pin header THT 1x04 2.54mm single row")
 		(property "Reference" "J3"
-			(at 2 -0.85 180)
+			(at 0.29 -2.57 180)
 			(layer "F.SilkS")
 			(effects
@@
 		(tags "capacitor")
 		(property "Reference" "C4"
-			(at 0 1.67 0)
+			(at 2.52 0.9 0)
 			(layer "F.SilkS")
 			(effects
@@
 	)
 	(zone
-		(net 20)
-		(net_name "/MISO")
+		(net 1)
+		(net_name "GND")
 		(layer "B.Cu")
 		(hatch edge 0.5)
@@
 		(filled_areas_thickness no)
 		(fill yes
-			(mode hatch)
 			(thermal_gap 0.5)
 			(thermal_bridge_width 0.5)
-			(hatch_thickness 1)
-			(hatch_gap 1.5)
-			(hatch_orientation 0)
-			(hatch_border_algorithm hatch_thickness)
-			(hatch_min_hole_area 0.3)
 		)
 		(polygon
@@
 		(filled_areas_thickness no)
 		(fill yes
-			(mode hatch)
 			(thermal_gap 0.5)
 			(thermal_bridge_width 0.5)
-			(hatch_thickness 1)
-			(hatch_gap 1.5)
-			(hatch_orientation 0)
-			(hatch_border_algorithm hatch_thickness)
-			(hatch_min_hole_area 0.3)
 		)
 		(polygon
